File: flip_pendant.kicad_pcb (KiCad board)
At the start: 4 copper layers, 34.4 x 34.4 mm, 264 parts, among them U1 RP2350_60QFN, U1 TPS3839A09DQNR, U2 TPS7A0215PDQNR, U3 MCP73832-2-MC, U5 BMA400, Y1 ABM8-272-T3

Commit message: clean up in2.cu
Routing:
- net GPIO5: track 87.1 -> 78.4 mm
- net GPIO2: track 80.0 -> 72.3 mm
- net GPIO7: track 80.2 -> 75.8 mm
- net GPIO3: track 65.5 -> 61.4 mm
- net GPIO8: track 89.8 -> 86.1 mm
- net GPIO1: track 82.1 -> 78.7 mm
- net GPIO6: track 79.2 -> 77.4 mm
- net GPIO18: track 59.7 -> 58.1 mm
- net GPIO9: track 66.0 -> 64.7 mm
- net GPIO4: track 74.0 -> 73.2 mm
- net GPIO10: track 77.0 -> 76.2 mm
